File: Hardware/OpenBook_Reader.brd (EAGLE design)
At the start: 170.2 x 111.2 mm, 103 parts, among them IC1 BD5229G-TR, IC4 XC6220A331MR-G, J1 FH34SRJ-24S-0.5SH_99_, J2 SAMACSYS_PARTS_USB4110-GF-A, J3 QWIIC_RIGHT_ANGLE, J4 112A-TAAR-R03_ATTEND, Q1 20V/4.2A/52mΩ/1.4W, Q2 20V/4.2A/52mΩ/1.4W, Q3 SI1308EDL-T1-GE3, U1 W25Q512JVEIQ, U2 ESP32-C6-WROOM-1-N8, U3 DS3231SN#, U4 MAX17048G+T10, U5 ESP32_WROVER_SPARKFUN-IC-POWE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

Commit message: Rezolvat Plan de Masa
Parts:
- removed TP6: TPTP20R, DeskAssistant v19 v1:TP20R
- added MISO: TPTP20R, DeskAssistant v19 v1:TP20R
- R10, R5, R6, R7, R8, R9: value (none) -> 10K
- renumbered TP1 to TX, TP10 to EPD_CS, TP11 to EPD_DC, TP12 to EPD_RST, TP13 to EPD_3V3_C, TP14 to VBUS, TP15 to INT_RTC, TP16 to 3V3, TP17 to EPD_3V3, TP2 to RX, TP3 to VBAT, TP4 to GND, TP5 to GND., TP7 to MOSI, TP8 to SCK, TP9 to EPD_BUSY
Connections:
- net MISO: now also MISO.TP; no longer TP6.TP
